File: fileAddressCounter.sch (KiCad schematic (older format))
At the start: 16 parts, among them U13 CD74AC161M, U14 CD74AC161M, U16 CD74AC161M, U17 CD74AC161M, U18 74AHC1G04, U19 CD74AC161M, U20 CD74AC161M, U38 74AHC1G04, U39 74AHC1G04

Commit message: Update materials list, begin to work on pcb
Parts:
- U13, U14, U16, U17, U19, U20: footprint (none) -> Package_SO:SOP-16_3.9x9.9mm_P1.27mm
- U18, U38, U39: footprint (none) -> Package_TO_SOT_SMD:SOT-23-5
Changed lines of the file:
@@
 F 0 "U18" H 10050 5850 50  0000 L CNN
 F 1 "74AHC1G04" H 10050 5750 50  0000 L CNN
-F 2 "" H 9950 5600 50  0001 C CNN
+F 2 "Package_TO_SOT_SMD:SOT-23-5" H 9950 5600 50  0001 C CNN
 F 3 "https://assets.nexperia.com/documents/data-sheet/74AHC_AHCT1G04.pdf" H 9950 5600 50  0001 C CNN
 	1    9950 5600
@@
 F 0 "U39" H 7800 5850 50  0000 L CNN
 F 1 "74AHC1G04" H 7800 5750 50  0000 L CNN
-F 2 "" H 7700 5600 50  0001 C CNN
+F 2 "Package_TO_SOT_SMD:SOT-23-5" H 7700 5600 50  0001 C CNN
 F 3 "https://assets.nexperia.com/documents/data-sheet/74AHC_AHCT1G04.pdf" H 7700 5600 50  0001 C CNN
 	1    7700 5600
@@
 F 0 "U38" H 6950 5850 50  0000 L CNN
 F 1 "74AHC1G04" H 6950 5750 50  0000 L CNN
-F 2 "" H 6850 5600 50  0001 C CNN
+F 2 "Package_TO_SOT_SMD:SOT-23-5" H 6850 5600 50  0001 C CNN
 F 3 "https://assets.nexperia.com/documents/data-sheet/74AHC_AHCT1G04.pdf" H 6850 5600 50  0001 C CNN
 	1    6850 5600
@@
 F 0 "U19" H 8350 2250 60  0000 C CNN
 F 1 "CD74AC161M" H 8550 2150 60  0000 C CNN
-F 2 "" H 7950 1950 60  0001 C CNN
+F 2 "Package_SO:SOP-16_3.9x9.9mm_P1.27mm" H 7950 1950 60  0001 C CNN
 F 3 "https://www.ti.com/lit/ds/symlink/cd74ac161.pdf" H 7950 1950 60  0001 C CNN
 	1    8100 1650
@@
 F 0 "U20" H 8350 4200 60  0000 C CNN
 F 1 "CD74AC161M" H 8550 4100 60  0000 C CNN
-F 2 "" H 7950 3900 60  0001 C CNN
+F 2 "Package_SO:SOP-16_3.9x9.9mm_P1.27mm" H 7950 3900 60  0001 C CNN
 F 3 "https://www.ti.com/lit/ds/symlink/cd74ac161.pdf" H 7950 3900 60  0001 C CNN
 	1    8100 3600
@@
 F 0 "U16" H 5500 2250 60  0000 C CNN
 F 1 "CD74AC161M" H 5700 2150 60  0000 C CNN
-F 2 "" H 5100 1950 60  0001 C CNN
+F 2 "Package_SO:SOP-16_3.9x9.9mm_P1.27mm" H 5100 1950 60  0001 C CNN
 F 3 "https://www.ti.com/lit/ds/symlink/cd74ac161.pdf" H 5100 1950 60  0001 C CNN
 	1    5250 1650
@@
 F 0 "U17" H 5500 4200 60  0000 C CNN
 F 1 "CD74AC161M" H 5700 4100 60  0000 C CNN
-F 2 "" H 5100 3900 60  0001 C CNN
+F 2 "Package_SO:SOP-16_3.9x9.9mm_P1.27mm" H 5100 3900 60  0001 C CNN
 F 3 "https://www.ti.com/lit/ds/symlink/cd74ac161.pdf" H 5100 3900 60  0001 C CNN
 	1    5250 3600
@@
 F 0 "U13" H 2650 2250 60  0000 C CNN
 F 1 "CD74AC161M" H 2850 2150 60  0000 C CNN
-F 2 "" H 2250 1950 60  0001 C CNN
+F 2 "Package_SO:SOP-16_3.9x9.9mm_P1.27mm" H 2250 1950 60  0001 C CNN
 F 3 "https://www.ti.com/lit/ds/symlink/cd74ac161.pdf" H 2250 1950 60  0001 C CNN
 	1    2400 1650
@@
 F 0 "U14" H 2650 4200 60  0000 C CNN
 F 1 "CD74AC161M" H 2850 4100 60  0000 C CNN
-F 2 "" H 2250 3900 60  0001 C CNN
+F 2 "Package_SO:SOP-16_3.9x9.9mm_P1.27mm" H 2250 3900 60  0001 C CNN
 F 3 "https://www.ti.com/lit/ds/symlink/cd74ac161.pdf" H 2250 3900 60  0001 C CNN
 	1    2400 3600
@@
 Text Label 4750 3350 2    60   ~ 0
 ~CLEAR
+$Comp
+L power:+3.3V #PWR0113
+U 1 1 5FB4F2DF
+P 2400 2850
+F 0 "#PWR0113" H 2400 2700 50  0001 C CNN
+F 1 "+3.3V" H 2350 3000 50  0000 C CNN
+F 2 "" H 2400 2850 50  0001 C CNN
+F 3 "" H 2400 2850 50  0001 C CNN
+	1    2400 2850
+	1    0    0    -1
+$EndComp
+$Comp
+L power:+3.3V #PWR0114
+U 1 1 5FB4F581
+P 2400 900
+F 0 "#PWR0114" H 2400 750 50  0001 C CNN
+F 1 "+3.3V" H 2350 1050 50  0000 C CNN
+F 2 "" H 2400 900 50  0001 C CNN
+F 3 "" H 2400 900 50  0001 C CNN
+	1    2400 900
+	1    0    0    -1
+$EndComp
+$Comp
+L power:+3.3V #PWR0121
+U 1 1 5FB4FC54
+P 5250 900
+F 0 "#PWR0121" H 5250 750 50  0001 C CNN
+F 1 "+3.3V" H 5200 1050 50  0000 C CNN
+F 2 "" H 5250 900 50  0001 C CNN
+F 3 "" H 5250 900 50  0001 C CNN
+	1    5250 900
+	1    0    0    -1
+$EndComp
+$Comp
+L power:+3.3V #PWR0122
+U 1 1 5FB500AA
+P 8100 900
+F 0 "#PWR0122" H 8100 750 50  0001 C CNN
+F 1 "+3.3V" H 8050 1050 50  0000 C CNN
+F 2 "" H 8100 900 50  0001 C CNN
+F 3 "" H 8100 900 50  0001 C CNN
+	1    8100 900
+	1    0    0    -1
+$EndComp
+$Comp
+L power:+3.3V #PWR0124
+U 1 1 5FB50551
+P 8100 2850
+F 0 "#PWR0124" H 8100 2700 50  0001 C CNN
+F 1 "+3.3V" H 8050 3000 50  0000 C CNN
+F 2 "" H 8100 2850 50  0001 C CNN
+F 3 "" H 8100 2850 50  0001 C CNN
+	1    8100 2850
+	1    0    0    -1
+$EndComp
+$Comp
+L power:+3.3V #PWR0168
+U 1 1 5FB50AC7
+P 5250 2850
+F 0 "#PWR0168" H 5250 2700 50  0001 C CNN
+F 1 "+3.3V" H 5200 3000 50  0000 C CNN
+F 2 "" H 5250 2850 50  0001 C CNN
+F 3 "" H 5250 2850 50  0001 C CNN
+	1    5250 2850
+	1    0    0    -1
+$EndComp
 Wire Bus Line
 	5450 6100 5450 7300
@@
 Wire Bus Line
 	1550 6100 1550 7300
-$Comp
-L power:+3.3V #PWR0113
-U 1 1 5FB4F2DF
-P 2400 2850
-F 0 "#PWR0113" H 2400 2700 50  0001 C CNN
-F 1 "+3.3V" H 2350 3000 50  0000 C CNN
-F 2 "" H 2400 2850 50  0001 C CNN
-F 3 "" H 2400 2850 50  0001 C CNN
-	1    2400 2850
-	1    0    0    -1
-$EndComp
-$Comp
-L power:+3.3V #PWR0114
-U 1 1 5FB4F581
-P 2400 900
-F 0 "#PWR0114" H 2400 750 50  0001 C CNN
-F 1 "+3.3V" H 2350 1050 50  0000 C CNN
-F 2 "" H 2400 900 50  0001 C CNN
-F 3 "" H 2400 900 50  0001 C CNN
-	1    2400 900
-	1    0    0    -1
-$EndComp
-$Comp
-L power:+3.3V #PWR0121
-U 1 1 5FB4FC54
-P 5250 900
-F 0 "#PWR0121" H 5250 750 50  0001 C CNN
-F 1 "+3.3V" H 5200 1050 50  0000 C CNN
-F 2 "" H 5250 900 50  0001 C CNN
-F 3 "" H 5250 900 50  0001 C CNN
-	1    5250 900
-	1    0    0    -1
-$EndComp
-$Comp
-L power:+3.3V #PWR0122
-U 1 1 5FB500AA
-P 8100 900
-F 0 "#PWR0122" H 8100 750 50  0001 C CNN
-F 1 "+3.3V" H 8050 1050 50  0000 C CNN
-F 2 "" H 8100 900 50  0001 C CNN
-F 3 "" H 8100 900 50  0001 C CNN
-	1    8100 900
-	1    0    0    -1
-$EndComp
-$Comp
-L power:+3.3V #PWR0124
-U 1 1 5FB50551
-P 8100 2850
-F 0 "#PWR0124" H 8100 2700 50  0001 C CNN
-F 1 "+3.3V" H 8050 3000 50  0000 C CNN
-F 2 "" H 8100 2850 50  0001 C CNN
-F 3 "" H 8100 2850 50  0001 C CNN
-	1    8100 2850
-	1    0    0    -1
-$EndComp
-$Comp
-L power:+3.3V #PWR0168
-U 1 1 5FB50AC7
-P 5250 2850
-F 0 "#PWR0168" H 5250 2700 50  0001 C CNN
-F 1 "+3.3V" H 5200 3000 50  0000 C CNN
-F 2 "" H 5250 2850 50  0001 C CNN
-F 3 "" H 5250 2850 50  0001 C CNN
-	1    5250 2850
-	1    0    0    -1
-$EndComp
 $EndSCHEMATC
