File: fileAddressExchanger.sch (KiCad schematic (older format))
At the start: 10 parts, among them U23 74CBTLV16212, U24 74CBTLV16212, U42 74AHC273, U43 74AHC273, U44 74AHC273

Commit message: Update materials list, begin to work on pcb
Parts:
- U23, U24: footprint (none) -> Package_SO:TSSOP-56_6.1x14mm_P0.5mm
Changed lines of the file:
@@
 F 0 "U23" H 4250 4150 50  0000 C CNN
 F 1 "74CBTLV16212" H 4450 4050 50  0000 C CNN
-F 2 "" H 4100 3300 50  0001 C CNN
+F 2 "Package_SO:TSSOP-56_6.1x14mm_P0.5mm" H 4100 3300 50  0001 C CNN
 F 3 "https://www.ti.com/lit/ds/symlink/sn74cbtlv16212.pdf" H 4100 3300 50  0001 C CNN
 	1    4100 2500
@@
 F 0 "U24" H 7300 4150 50  0000 C CNN
 F 1 "74CBTLV16212" H 7500 4050 50  0000 C CNN
-F 2 "" H 7150 3300 50  0001 C CNN
+F 2 "Package_SO:TSSOP-56_6.1x14mm_P0.5mm" H 7150 3300 50  0001 C CNN
 F 3 "https://www.ti.com/lit/ds/symlink/sn74cbtlv16212.pdf" H 7150 3300 50  0001 C CNN
 	1    7150 2500
