File: fileClockGenerator.sch (KiCad schematic (older format))
At the start: 16 parts, among them U26 SN74LV393A, U27 SN74LV393A, U28 CD74AC151, U29 CD74AC151, U30 74AHC1G32, U31 CD74AC151, U4 74AHC273, X1 ECS-2200BX-500

Commit message: Update materials list, begin to work on pcb
Parts:
- C11: footprint Capacitor_SMD:C_0805_2012Metric -> Capacitor_SMD:C_1206_3216Metric
- R6: footprint (none) -> Resistor_SMD:R_0805_2012Metric
- U26, U27: footprint (none) -> Package_SO:SOIC-14_3.9x8.7mm_P1.27mm
- U28, U29, U31: footprint (none) -> Package_SO:SOP-16_3.9x9.9mm_P1.27mm
- U30: footprint (none) -> Package_TO_SOT_SMD:SOT-23-5
Changed lines of the file:
@@
 F 0 "C11" H 1425 2100 50  0000 L CNN
 F 1 "100nF" H 1425 1900 50  0000 L CNN
-F 2 "Capacitor_SMD:C_0805_2012Metric" H 1438 1850 50  0001 C CNN
+F 2 "Capacitor_SMD:C_1206_3216Metric" H 1438 1850 50  0001 C CNN
 F 3 "" H 1400 2000 50  0001 C CNN
 	1    1400 2000
@@
 F 0 "R6" H 2320 2096 50  0000 L CNN
 F 1 "10k" H 2320 2005 50  0000 L CNN
-F 2 "" V 2180 2050 50  0001 C CNN
+F 2 "Resistor_SMD:R_0805_2012Metric" V 2180 2050 50  0001 C CNN
 F 3 "~" H 2250 2050 50  0001 C CNN
 	1    2250 2050
@@
 F 0 "U26" H 5100 2150 60  0000 C CNN
 F 1 "SN74LV393A" H 5300 2050 60  0000 C CNN
-F 2 "" H 4800 1850 60  0001 C CNN
+F 2 "Package_SO:SOIC-14_3.9x8.7mm_P1.27mm" H 4800 1850 60  0001 C CNN
 F 3 "https://www.ti.com/lit/ds/symlink/sn74lv393a-q1.pdf" H 4800 1850 60  0001 C CNN
 	1    4950 1550
@@
 F 0 "U27" H 5100 4500 60  0000 C CNN
 F 1 "SN74LV393A" H 5300 4400 60  0000 C CNN
-F 2 "" H 4800 4200 60  0001 C CNN
+F 2 "Package_SO:SOIC-14_3.9x8.7mm_P1.27mm" H 4800 4200 60  0001 C CNN
 F 3 "https://www.ti.com/lit/ds/symlink/sn74lv393a-q1.pdf" H 4800 4200 60  0001 C CNN
 	1    4950 3900
@@
 F 0 "U28" H 8200 2650 50  0000 C CNN
 F 1 "CD74AC151" H 8350 2550 50  0000 C CNN
-F 2 "" H 8050 1800 50  0001 C CNN
+F 2 "Package_SO:SOP-16_3.9x9.9mm_P1.27mm" H 8050 1800 50  0001 C CNN
 F 3 "https://www.ti.com/lit/ds/symlink/cd74ac151.pdf" H 8050 1800 50  0001 C CNN
 	1    8050 1800
@@
 F 0 "U29" H 8200 5200 50  0000 C CNN
 F 1 "CD74AC151" H 8350 5100 50  0000 C CNN
-F 2 "" H 8050 4350 50  0001 C CNN
+F 2 "Package_SO:SOP-16_3.9x9.9mm_P1.27mm" H 8050 4350 50  0001 C CNN
 F 3 "https://www.ti.com/lit/ds/symlink/cd74ac151.pdf" H 8050 4350 50  0001 C CNN
 	1    8050 4350
@@
 F 0 "U31" H 10250 3250 50  0000 C CNN
 F 1 "CD74AC151" H 10400 3150 50  0000 C CNN
-F 2 "" H 10100 2400 50  0001 C CNN
+F 2 "Package_SO:SOP-16_3.9x9.9mm_P1.27mm" H 10100 2400 50  0001 C CNN
 F 3 "https://www.ti.com/lit/ds/symlink/cd74ac151.pdf" H 10100 2400 50  0001 C CNN
 	1    10100 2400
@@
 F 0 "U30" H 9600 5750 50  0000 L CNN
 F 1 "74AHC1G32" H 9600 5650 50  0000 L CNN
-F 2 "" H 9500 5500 50  0001 C CNN
+F 2 "Package_TO_SOT_SMD:SOT-23-5" H 9500 5500 50  0001 C CNN
 F 3 "http://www.ti.com/lit/sg/scyt129e/scyt129e.pdf" H 9500 5500 50  0001 C CNN
 	1    9500 5500
