File: fileClockGenerator.sch (KiCad schematic (older format))
At the start: 16 parts, among them U26 SN74LV393A, U27 SN74LV393A, U28 CD74AC151, U29 CD74AC151, U30 74AHC1G32, U31 CD74AC151, U4 74AHC273, X1 ECS-2200BX-500

Commit message: Set every capacitor size to 0805
Parts:
- C11: footprint Capacitor_SMD:C_1206_3216Metric -> Capacitor_SMD:C_0805_2012Metric
Changed lines of the file:
@@
 F 0 "C11" H 1425 2100 50  0000 L CNN
 F 1 "100nF" H 1425 1900 50  0000 L CNN
-F 2 "Capacitor_SMD:C_1206_3216Metric" H 1438 1850 50  0001 C CNN
+F 2 "Capacitor_SMD:C_0805_2012Metric" H 1438 1850 50  0001 C CNN
 F 3 "" H 1400 2000 50  0001 C CNN
 	1    1400 2000
