File: fileClockGenerator.sch (KiCad schematic (older format))
At the start: 16 parts, among them U26 SN74LV393A, U27 SN74LV393A, U28 CD74AC151, U29 CD74AC151, U30 74AHC1G32, U31 CD74AC151, U4 74AHC273, X1 ECS-2200BX-500

Commit message: V5.1 (#15)
* Remove compatibility for 5.0, 4.x and add 5.1+

* Fix switched pins on SN74LV393A #7

* Removed capacitor on 12V #11

* Add/Modify power decoupling capacitor #10

* Removing ADDSCR_CLK delay #9

* Schematics : set version 5.1, 2021 copyright and publish date

* Put non-electrolytic capacitor #10

* Set every capacitor size to 0805

* Add new footprint for J7 TE_3-641124-6 #6

* Schematic : set pinHeader on J12 #4

* Netlist, apply change to board, clean track, #6 #4 #12 #10

* Set version to 5.1, 2021 copyright and date, replace the missing QRcode

* Back the MM1 connectors #8

* Replace capacitor for U22 U23 U24 #13

* Better decoupling

* Increase version, year to 2021, clear status

* Precise the molex connector for power supply

* First step, import ses

* Clean bottom layer

* #14 Set the BWRITE2 bus instead of BWRITE1 on U12

* netlist, redo autorouting and cleaning

* use shields.io for colored badge

* Update gerbert files

* Changelog, updated BOM

* Small revision on blockDiagram

* Update README.md

* exporting pcb in pdf

* 3D images, diagram.png

* Update schematics pdf

* redo wavedrom_24bitsCounter
Parts:
- C11: footprint Capacitor_SMD:C_1206_3216Metric -> Capacitor_SMD:C_0805_2012Metric
Changed lines of the file:
@@
 Sheet 4 10
 Title "GCM"
-Date "2020-11-23"
-Rev "V5.0"
+Date "2021-02-16"
+Rev "V5.1"
 Comp "Guillaume Guillet"
-Comment1 "Copyright Guillaume Guillet 2020"
+Comment1 "Copyright Guillaume Guillet 2021"
 Comment2 "Licensed under CERN-OHL-W v2 or later"
 Comment3 ""
@@
 F 0 "C11" H 1425 2100 50  0000 L CNN
 F 1 "100nF" H 1425 1900 50  0000 L CNN
-F 2 "Capacitor_SMD:C_1206_3216Metric" H 1438 1850 50  0001 C CNN
+F 2 "Capacitor_SMD:C_0805_2012Metric" H 1438 1850 50  0001 C CNN
 F 3 "" H 1400 2000 50  0001 C CNN
 	1    1400 2000
@@
 U 1 1 5FDD1821
 P 4950 1550
+AR Path="/5FDD1821" Ref="U26"  Part="1"
+AR Path="/5B3313A4/5FDD1821" Ref="U26"  Part="1"
 F 0 "U26" H 5100 2150 60  0000 C CNN
 F 1 "SN74LV393A" H 5300 2050 60  0000 C CNN
@@
 U 1 1 5FDD314D
 P 4950 3900
+AR Path="/5FDD314D" Ref="U27"  Part="1"
+AR Path="/5B3313A4/5FDD314D" Ref="U27"  Part="1"
 F 0 "U27" H 5100 4500 60  0000 C CNN
 F 1 "SN74LV393A" H 5300 4400 60  0000 C CNN
