File: fileConnector.sch (KiCad schematic (older format))
At the start: 13 parts, among them J6 TE_Eurocard_96pole, J9 Conn_01x02, U8 74AHC244, U9 74AHC244

Commit message: Update materials list, begin to work on pcb
Parts:
- H1, H2, H3, H4: footprint (none) -> MountingHole:MountingHole_3mm
Changed lines of the file:
@@
 F 0 "H1" H 6800 3096 50  0000 L CNN
 F 1 "MountingHole_3mm" H 6800 3005 50  0000 L CNN
-F 2 "" H 6700 3050 50  0001 C CNN
+F 2 "MountingHole:MountingHole_3mm" H 6700 3050 50  0001 C CNN
 F 3 "~" H 6700 3050 50  0001 C CNN
 	1    6700 3050
@@
 F 0 "H2" H 7850 3096 50  0000 L CNN
 F 1 "MountingHole_3mm" H 7850 3005 50  0000 L CNN
-F 2 "" H 7750 3050 50  0001 C CNN
+F 2 "MountingHole:MountingHole_3mm" H 7750 3050 50  0001 C CNN
 F 3 "~" H 7750 3050 50  0001 C CNN
 	1    7750 3050
@@
 F 0 "H3" H 6800 3596 50  0000 L CNN
 F 1 "MountingHole_3mm" H 6800 3505 50  0000 L CNN
-F 2 "" H 6700 3550 50  0001 C CNN
+F 2 "MountingHole:MountingHole_3mm" H 6700 3550 50  0001 C CNN
 F 3 "~" H 6700 3550 50  0001 C CNN
 	1    6700 3550
@@
 F 0 "H4" H 7850 3596 50  0000 L CNN
 F 1 "MountingHole_3mm" H 7850 3505 50  0000 L CNN
-F 2 "" H 7750 3550 50  0001 C CNN
+F 2 "MountingHole:MountingHole_3mm" H 7750 3550 50  0001 C CNN
 F 3 "~" H 7750 3550 50  0001 C CNN
 	1    7750 3550
