File: fileMemoryController.sch (KiCad schematic (older format))
At the start: 10 parts, among them U10 74LVC1G74, U12 74AHC244, U15 74AHC1G04, U21 74AHC244, U22 74CBTLV16212

Commit message: see CHANGELOG
Parts:
- removed U15: 74AHC1G04, symbol Custom:74AHC1G04
- removed U21: 74AHC244, Package_SO:SOIC-20W_7.5x12.8mm_P1.27mm, symbol 74xx:74AHC244
- removed U22: 74CBTLV16212, Package_SO:TSSOP-56_6.1x14mm_P0.5mm, symbol Custom:74CBTLV16212
- added C52: 10nF, Capacitor_SMD:C_0805_2012Metric, symbol Device:C
- added U15: 74AHCT1G04, symbol Custom:74AHCT1G04
- added U21: 74AHCT244, symbol 74xx:74AHCT244
- added U22: 74CBTLV16212, symbol 74xx:74CBTLV16212
- added U40: 74AHC273, Package_SO:SOIC-20W_7.5x12.8mm_P1.27mm, symbol 74xx:74AHC273
- added U41: 74AHC1G04, symbol Custom:74AHC1G04
Connections:
- net +3V3: now also C23.2, C28.2, U10.7 (~PRE), U10.8 (VCC), U12.20 (VCC), C52.2, U22.17 (VCC), U22.23 (10A1), U22.55 (S2), U22.56 (S1), U40.20 (VCC), U41.5 (VCC)
- net +5V: now also U15.5 (VCC), U21.20 (VCC); no longer C23.2, C28.2, U10.7 (~PRE), U10.8 (VCC), U12.20 (VCC)
- net BDATASRC_0: now also U22.2 (1A1)
- net BDATASRC_1: now also U22.4 (2A1)
- net BDATASRC_2: now also U22.6 (3A1)
- net BDATASRC_3: now also U22.9 (4A1)
- net BDATASRC_4: now also U22.11 (5A1)
- net BDATASRC_5: now also U22.13 (6A1)
- net BDATASRC_6: now also U22.15 (7A1)
- net BDATASRC_7: now also U22.18 (8A1)
- net BREAD1_0: now also U21.18 (1Y0)
- net BREAD1_1: now also U21.16 (1Y1)
- net BREAD1_2: now also U21.14 (1Y2)
- net BREAD1_3: now also U21.12 (1Y3)
- net BREAD1_4: now also U21.3 (2Y0)
- net BREAD1_5: now also U21.5 (2Y1)
- net BREAD1_6: now also U21.7 (2Y2)
- net BREAD1_7: now also U21.9 (2Y3)
- net BWRITE1_0: now also U40.3 (D0)
- net BWRITE1_1: now also U40.4 (D1)
- net BWRITE1_2: now also U40.7 (D2)
- net BWRITE1_3: now also U40.8 (D3)
- net BWRITE1_4: now also U40.13 (D4)
- net BWRITE1_5: now also U40.14 (D5)
- net GND: now also C52.1, U15.3 (GND), U21.10 (GND), U22.19 (GND), U22.21 (9A1), U22.25 (11A1), U22.27 (12A1), U22.28 (12A2), U22.38 (GND), U22.49 (GND), U22.8 (GND), U40.10 (GND), U40.17 (D6), U40.18 (D7), U41.3 (GND)
- net MEM1DATA_0: now also U22.54 (1B1)
- net MEM1DATA_1: now also U22.52 (2B1)
- net MEM1DATA_2: now also U22.50 (3B1)
- net MEM1DATA_3: now also U22.47 (4B1)
- net MEM1DATA_4: now also U22.45 (5B1)
- net MEM1DATA_5: now also U22.43 (6B1)
- net MEM1DATA_6: now also U22.41 (7B1)
- net MEM1DATA_7: now also U22.39 (8B1)
- net MEM1_~CE: now also U22.36 (9B1)
- net MEM1_~OE: now also U22.32 (11B1)
- net MEM1_~WE: now also U22.34 (10B1)
- net MEM2DATA_0: now also U22.53 (1B2)
- net MEM2DATA_1: now also U22.51 (2B2)
- net MEM2DATA_2: now also U22.48 (3B2)
- net MEM2DATA_3: now also U22.46 (4B2)
- net MEM2DATA_4: now also U22.44 (5B2)
- net MEM2DATA_5: now also U22.42 (6B2)
- net MEM2DATA_6: now also U22.40 (7B2)
- net MEM2DATA_7: now also U22.37 (8B2)
- net MEM2_~CE: now also U22.35 (9B2)
- net MEM2_~OE: now also U22.31 (11B2)
- net MEM2_~WE: now also U22.33 (10B2)
- net SRC_SELECTION: now also U22.1 (S0)
- net USER_RW_0: now also U21.2 (1A0), U22.3 (1A2)
- net USER_RW_1: now also U21.4 (1A1), U22.5 (2A2)
- net USER_RW_2: now also U21.6 (1A2), U22.7 (3A2)
- net USER_RW_3: now also U21.8 (1A3), U22.10 (4A2)
- net USER_RW_4: now also U21.17 (2A0), U22.12 (5A2)
- net USER_RW_5: now also U21.15 (2A1), U22.14 (6A2)
- net USER_RW_6: now also U21.13 (2A2), U22.16 (7A2)
- net USER_RW_7: now also U21.11 (2A3), U22.20 (8A2)
- net SRCSET_CLK renamed CLK_MODULE_SRCSET
- net ~CS~_WRITE_MODE renamed USER_OE
- net USER_OE: now also U15.4
- net ~RESET_CLK renamed ~RESET
- net ~RESET: now also U40.1 (~Mr)
- new net CLK_MODULE_MEMUSER: U40.11 (Cp)
- new net USER_ADDRESS_CLK_0: U40.9 (Q3)
- new net USER_ADDRESS_CLK_1: U40.12 (Q4)
- new net USER_ADDRESS_CLK_2: U40.15 (Q5)
- new net USER_CE: U40.2 (Q0), U41.2
- new net USER_~CE: U22.22 (9A2), U41.4
- new net USER_~OE: U15.2, U22.26 (11A2), U40.6 (Q2)
- new net USER_~WE: U22.24 (10A2), U40.5 (Q1)
- new net ~CS_MODULE_MEMUSER: U21.1 (1OE), U21.19 (2OE)
- no-connect marks 3 -> 5
Other:
- moved on the sheet: C23, C30, U10

Commit message: Update materials list, begin to work on pcb
Parts:
- U10: footprint (none) -> Package_SO:SSOP-8_2.95x2.8mm_P0.65mm
- U15, U41: footprint (none) -> Package_TO_SOT_SMD:SOT-23-5
- U21: footprint (none) -> Package_SO:SOIC-20W_7.5x12.8mm_P1.27mm
- U22: footprint (none) -> Package_SO:TSSOP-56_6.1x14mm_P0.5mm
Changed lines of the file:
@@
 F 0 "U10" H 1950 1500 50  0000 L CNN
 F 1 "74LVC1G74" H 1950 1400 50  0000 L CNN
-F 2 "" H 1800 1150 50  0001 C CNN
+F 2 "Package_SO:SSOP-8_2.95x2.8mm_P0.65mm" H 1800 1150 50  0001 C CNN
 F 3 "http://www.ti.com/lit/sg/scyt129e/scyt129e.pdf" H 1800 1150 50  0001 C CNN
 	1    1800 1150
@@
 F 0 "U21" H 5500 7350 50  0000 C CNN
 F 1 "74AHCT244" H 5650 7250 50  0000 C CNN
-F 2 "" H 5400 6600 50  0001 C CNN
+F 2 "Package_SO:SOIC-20W_7.5x12.8mm_P1.27mm" H 5400 6600 50  0001 C CNN
 F 3 "https://assets.nexperia.com/documents/data-sheet/74AHC_AHCT244.pdf" H 5400 6600 50  0001 C CNN
 	1    5400 6600
@@
 F 0 "U15" H 8150 6250 50  0000 L CNN
 F 1 "74AHCT1G04" H 8150 6150 50  0000 L CNN
-F 2 "" H 8050 6000 50  0001 C CNN
+F 2 "Package_TO_SOT_SMD:SOT-23-5" H 8050 6000 50  0001 C CNN
 F 3 "https://assets.nexperia.com/documents/data-sheet/74AHC_AHCT1G04.pdf" H 8050 6000 50  0001 C CNN
 	1    8050 6000
@@
 F 0 "U41" H 8150 5250 50  0000 L CNN
 F 1 "74AHC1G04" H 8150 5150 50  0000 L CNN
-F 2 "" H 8050 5000 50  0001 C CNN
+F 2 "Package_TO_SOT_SMD:SOT-23-5" H 8050 5000 50  0001 C CNN
 F 3 "https://assets.nexperia.com/documents/data-sheet/74AHC_AHCT1G04.pdf" H 8050 5000 50  0001 C CNN
 	1    8050 5000
@@
 F 0 "U22" H 8500 4150 50  0000 C CNN
 F 1 "74CBTLV16212" H 8700 4050 50  0000 C CNN
-F 2 "" H 8350 3300 50  0001 C CNN
+F 2 "Package_SO:TSSOP-56_6.1x14mm_P0.5mm" H 8350 3300 50  0001 C CNN
 F 3 "https://www.ti.com/lit/ds/symlink/sn74cbtlv16212.pdf" H 8350 3300 50  0001 C CNN
 	1    8350 2500
@@
 Wire Wire Line
 	7150 3900 7150 4300
+Connection ~ 7150 3900
 Wire Bus Line
 	10000 4050 10000 4850
@@
 Wire Bus Line
 	1500 6800 1500 7600
-Connection ~ 7150 3900
 $EndSCHEMATC
