File: filePClockGenerator.sch (KiCad schematic (older format))
At the start: 12 parts, among them U32 74AHC273, U33 SN74LV393A, U34 SN74LV393A, U35 CD74AC151, U36 CD74AC151, U37 CD74AC151

Commit message: Update materials list, begin to work on pcb
Parts:
- U33, U34: footprint (none) -> Package_SO:SOIC-14_3.9x8.7mm_P1.27mm
- U35, U36, U37: footprint (none) -> Package_SO:SOP-16_3.9x9.9mm_P1.27mm
Changed lines of the file:
@@
 F 0 "U33" H 5000 2250 60  0000 C CNN
 F 1 "SN74LV393A" H 5200 2150 60  0000 C CNN
-F 2 "" H 4700 1950 60  0001 C CNN
+F 2 "Package_SO:SOIC-14_3.9x8.7mm_P1.27mm" H 4700 1950 60  0001 C CNN
 F 3 "https://www.ti.com/lit/ds/symlink/sn74lv393a-q1.pdf" H 4700 1950 60  0001 C CNN
 	1    4850 1650
@@
 F 0 "U34" H 5000 4600 60  0000 C CNN
 F 1 "SN74LV393A" H 5200 4500 60  0000 C CNN
-F 2 "" H 4700 4300 60  0001 C CNN
+F 2 "Package_SO:SOIC-14_3.9x8.7mm_P1.27mm" H 4700 4300 60  0001 C CNN
 F 3 "https://www.ti.com/lit/ds/symlink/sn74lv393a-q1.pdf" H 4700 4300 60  0001 C CNN
 	1    4850 4000
@@
 F 0 "U35" H 8100 2750 50  0000 C CNN
 F 1 "CD74AC151" H 8250 2650 50  0000 C CNN
-F 2 "" H 7950 1900 50  0001 C CNN
+F 2 "Package_SO:SOP-16_3.9x9.9mm_P1.27mm" H 7950 1900 50  0001 C CNN
 F 3 "https://www.ti.com/lit/ds/symlink/cd74ac151.pdf" H 7950 1900 50  0001 C CNN
 	1    7950 1900
@@
 F 0 "U36" H 8100 5300 50  0000 C CNN
 F 1 "CD74AC151" H 8250 5200 50  0000 C CNN
-F 2 "" H 7950 4450 50  0001 C CNN
+F 2 "Package_SO:SOP-16_3.9x9.9mm_P1.27mm" H 7950 4450 50  0001 C CNN
 F 3 "https://www.ti.com/lit/ds/symlink/cd74ac151.pdf" H 7950 4450 50  0001 C CNN
 	1    7950 4450
@@
 F 0 "U37" H 10150 3350 50  0000 C CNN
 F 1 "CD74AC151" H 10300 3250 50  0000 C CNN
-F 2 "" H 10000 2500 50  0001 C CNN
+F 2 "Package_SO:SOP-16_3.9x9.9mm_P1.27mm" H 10000 2500 50  0001 C CNN
 F 3 "https://www.ti.com/lit/ds/symlink/cd74ac151.pdf" H 10000 2500 50  0001 C CNN
 	1    10000 2500
