File: filePeripherals.sch (KiCad schematic (older format))
At the start: 18 parts, among them J2 5-5530843-4, J3 5-5530843-4, J4 5-5530843-4, J5 5-5530843-4, U6 CD74AC238, U7 74AHC138

Commit message: see CHANGELOG
Parts:
- J2, J3, J4, J5: value 5-5530843-4 -> PP1_receptacle_TE_5-5530843-4
Connections:
- net BPCS_0: now also U6.1 (A0); no longer U6.4 (~G2A)
- net BPCS_1: now also U6.2 (A1); no longer U6.5 (~G2B)
- net BPCS_2: now also U6.3 (A2); no longer U6.6 (G1)
- net GND: now also U6.4 (~G2A), U6.5 (~G2B); no longer U6.1 (A0), U6.2 (A1)
- net PERIPHERAL_CLK: now also U6.6 (G1); no longer U6.3 (A2)
- net GLOBAL_CLK renamed P_CLK

Commit message: Update materials list, begin to work on pcb
Parts:
- J2, J3, J4, J5: footprint Eurocard:SHDR40W89P485X254_2X20_5740X935X1562P -> TE_5-5530843-4:TE_5-5530843-4
- U6: footprint (none) -> Package_SO:SOP-16_3.9x9.9mm_P1.27mm
Changed lines of the file:
@@
 F 0 "J2" H 3800 2950 50  0000 C CNN
 F 1 "PP1_receptacle_TE_5-5530843-4" H 3800 766 50  0000 C CNN
-F 2 "Eurocard:SHDR40W89P485X254_2X20_5740X935X1562P" H 3750 1900 50  0001 C CNN
+F 2 "TE_5-5530843-4:TE_5-5530843-4" H 3750 1900 50  0001 C CNN
 F 3 "~" H 3750 1900 50  0001 C CNN
 	1    3750 1900
@@
 F 0 "J4" H 5800 2950 50  0000 C CNN
 F 1 "PP1_receptacle_TE_5-5530843-4" H 5800 766 50  0000 C CNN
-F 2 "Eurocard:SHDR40W89P485X254_2X20_5740X935X1562P" H 5750 1900 50  0001 C CNN
+F 2 "TE_5-5530843-4:TE_5-5530843-4" H 5750 1900 50  0001 C CNN
 F 3 "~" H 5750 1900 50  0001 C CNN
 	1    5750 1900
@@
 F 0 "J3" H 3800 5450 50  0000 C CNN
 F 1 "PP1_receptacle_TE_5-5530843-4" H 3800 3266 50  0000 C CNN
-F 2 "Eurocard:SHDR40W89P485X254_2X20_5740X935X1562P" H 3750 4400 50  0001 C CNN
+F 2 "TE_5-5530843-4:TE_5-5530843-4" H 3750 4400 50  0001 C CNN
 F 3 "~" H 3750 4400 50  0001 C CNN
 	1    3750 4400
@@
 F 0 "J5" H 5800 5450 50  0000 C CNN
 F 1 "PP1_receptacle_TE_5-5530843-4" H 5800 3266 50  0000 C CNN
-F 2 "Eurocard:SHDR40W89P485X254_2X20_5740X935X1562P" H 5750 4400 50  0001 C CNN
+F 2 "TE_5-5530843-4:TE_5-5530843-4" H 5750 4400 50  0001 C CNN
 F 3 "~" H 5750 4400 50  0001 C CNN
 	1    5750 4400
@@
 F 0 "U6" H 2150 7250 50  0000 C CNN
 F 1 "CD74AC238" H 2300 7150 50  0000 C CNN
-F 2 "" H 2050 6800 50  0001 C CNN
+F 2 "Package_SO:SOP-16_3.9x9.9mm_P1.27mm" H 2050 6800 50  0001 C CNN
 F 3 "" H 2050 6800 50  0001 C CNN
 	1    2050 6700
