File: fileMemorySlot2.sch (KiCad schematic (older format))
At the start: 4 parts, among them J13 Conn_01x10, J8 5530843-2

Commit message: see CHANGELOG
Parts:
- J13: value Conn_01x10 -> MM1_addressExtension
- J8: value 5530843-2 -> MM1_receptacle_5530843-2
Connections:
- net MEM_ADD_0 renamed MEMADDRESS_0
- net MEM_ADD_1 renamed MEMADDRESS_1
- net MEM_ADD_10 renamed MEMADDRESS_10
- net MEM_ADD_11 renamed MEMADDRESS_11
- net MEM_ADD_12 renamed MEMADDRESS_12
- net MEM_ADD_13 renamed MEMADDRESS_13
- net MEM_ADD_14 renamed MEMADDRESS_14
- net MEM_ADD_15 renamed MEMADDRESS_15
- net MEM_ADD_16 renamed MEMADDRESS_16
- net MEM_ADD_17 renamed MEMADDRESS_17
- net MEM_ADD_18 renamed MEMADDRESS_18
- net MEM_ADD_19 renamed MEMADDRESS_19
- net MEM_ADD_2 renamed MEMADDRESS_2
- net MEM_ADD_20 renamed MEMADDRESS_20
- net MEM_ADD_21 renamed MEMADDRESS_21
- net MEM_ADD_22 renamed MEMADDRESS_22
- net MEM_ADD_23 renamed MEMADDRESS_23
- net MEM_ADD_3 renamed MEMADDRESS_3
- net MEM_ADD_4 renamed MEMADDRESS_4
- net MEM_ADD_5 renamed MEMADDRESS_5
- net MEM_ADD_6 renamed MEMADDRESS_6
- net MEM_ADD_7 renamed MEMADDRESS_7
- net MEM_ADD_8 renamed MEMADDRESS_8
- net MEM_ADD_9 renamed MEMADDRESS_9
- net MEM_FEEDBACK renamed MEMFEEDBACK
Other:
- note added: "Address extension"
- note added: "MM1 slot"
- note removed: "Connector 5530843-2 TE connectivity"
- moved on the sheet: C33, C34, J11, J13

Commit message: First pass on the PCB
Parts:
- J13: footprint Connector_Multicomp:Multicomp_MC9A12-1034_2x05_P2.54mm_Vertical -> Connector_IDC:IDC-Header_2x05_P2.54mm_Vertical
Changed lines of the file:
@@
 F 0 "J13" H 10218 1825 50  0000 C CNN
 F 1 "MM1_addressExtension" H 10218 1916 50  0000 C CNN
-F 2 "Connector_Multicomp:Multicomp_MC9A12-1034_2x05_P2.54mm_Vertical" H 10300 2550 50  0001 C CNN
+F 2 "Connector_IDC:IDC-Header_2x05_P2.54mm_Vertical" H 10300 2550 50  0001 C CNN
 F 3 "~" H 10300 2550 50  0001 C CNN
 	1    10300 2550
