File: Project_GCM.kicad_pcb (KiCad board)
At the start: 4 copper layers, 203 x 116 mm, 126 parts, among them J1 PowerSupply, J10 MM1_addressExtension, J11 MM1_receptacle_5530843-2, J12 DEBUG_BUSES, J13 MM1_addressExtension, J2 PP1_receptacle_TE_5-5530843-4, J3 PP1_receptacle_TE_5-5530843-4, J4 PP1_receptacle_TE_5-5530843-4, J5 PP1_receptacle_TE_5-5530843-4, J6 TE_Eurocard_96pole, J7 3-641124-6, J8 MM1_receptacle_5530843-2, J9 Conn_01x02, U1 LM810, U10 74LVC1G74, U11 74AHC1G04, U12 74AHC244, U13 CD74AC161M, U14 CD74AC161M, U15 74AHCT1G04, U16 CD74AC161M, U17 CD74AC161M, U18 74AHC1G04, U19 CD74AC161M, U2 LTC6994xS6-1, U20 CD74AC161M, U21 74AHCT244, U22 74CBTLV16212, U23 74CBTLV16212, U24 74CBTLV16212, U25 74AHC1G32, U26 SN74LV393A, U27 SN74LV393A, U28 CD74AC151, U29 CD74AC151, U3 74AHC1G32, U30 74AHC1G32, U31 CD74AC151, U32 74AHC273, U33 SN74LV393A, U34 SN74LV393A, U35 CD74AC151, U36 CD74AC151, U37 CD74AC151, U38 74AHC1G04, U39 74AHC1G04, U4 74AHC273, U40 74AHC273, U41 74AHC1G04, U42 74AHC273, U43 74AHC273, U44 74AHC273, U5 74AHC1G04, U6 CD74AC238, U7 74AHC138, U8 74AHC244, U9 74AHC244, X1 ECS-2200BX-500

Commit message: Add QRcode
Parts:
- added G***: LOGO, QRCode:QRCode, B.Cu at (249.1, 74.2)

Commit message: First generation of gerbert files
Routing:
- net GND: track 1475.7 -> 1447.7 mm
Other:
- net class Power added: clearance 0.2, trace_width 0.25, via_dia 0.55, via_drill 0.3
- net class Volt removed
- rule pad_to_mask_clearance: 0.2 -> 0
